Commit message: Make SHASTA pip-installable with a headless demo

File: shasta/assets/vehicles/arial_vehicle_abstract.urdf (robot description, URDF)
Before this commit: robot environment, 1 links, 0 joints
Links:
- removed link buildings
- added link base, mass 0.2; visual sphere radius=0.75

File: shasta/assets/vehicles/ground_vehicle_abstract.urdf (robot description, URDF)
Before this commit: robot environment, 1 links, 0 joints
Links:
- removed link buildings
- added link base_link, mass 1; visual box size=0.65 0.65 0.65

File: shasta/assets/vehicles/ground_vehicle_detailed.urdf (robot description, URDF)
Before this commit: robot environment, 1 links, 0 joints
Links:
- removed link buildings
- added link base_link, mass 1; collision box size=0.75 0.75 0.75; visual mesh filename=meshes/ugv.obj scale=0.025 0.025 0.025
